Commit message: Add SDF filea and Gazebo config

File: thor_gazebo/urdf/thor_urdf.xacro (robot description, xacro)
@@ -218,5 +218,5 @@
         </inertial>
     </link>
-    <joint name="joint_hand_finger_left" type="prismatic">
+    <!--joint name="joint_hand_finger_left" type="prismatic">
         <parent link="link_hand" />
         <child link="link_finger_left" />
@@ -276,5 +276,5 @@
             <inertia ixx="3358780.25" iyy="627437.875" izz="3410634.5" ixy="-145110.265625" ixz="93.539124" iyz="1280.361816" />
         </inertial>
-    </link>
+    </link-->
     <gazebo>
         <plugin filename="ignition-gazebo-joint-state-publisher-system" name="ignition::gazebo::systems::JointStatePublisher">
