Commit message: Thor Control Gazebo Classic

File: thor_description/urdf/thor_urdf.xacro (robot description, xacro)
@@ -232,5 +232,5 @@
         <axis xyz="0.5547 0.8321 0"/>
         <limit effort="100" lower="0.0" upper="0.06" velocity="10" />
-        <mimic joint="joint_hand_finger_left" />
+        <mimic joint="joint_hand_finger_left" multiplier="1.0" offset="0"/>
         <dynamics damping="0.3" friction="0.5" />
     </joint>
@@ -277,53 +277,3 @@
         </inertial>
     </link>
-    <gazebo>
-        <plugin filename="ignition-gazebo-joint-state-publisher-system" name="ignition::gazebo::systems::JointStatePublisher">
-            <topic>joint_states</topic>
-        </plugin>
-    </gazebo>
-    <gazebo>
-        <plugin filename="ignition-gazebo-joint-position-controller-system" name="ignition::gazebo::systems::JointPositionController">
-            <joint_name>joint_base_art1_yaw</joint_name>
-        </plugin>
-    </gazebo>
-    <gazebo>
-        <plugin filename="ignition-gazebo-joint-position-controller-system" name="ignition::gazebo::systems::JointPositionController">
-            <joint_name>joint_art1_art2_pitch</joint_name>
-        </plugin>
-    </gazebo>
-    <gazebo>
-        <plugin filename="ignition-gazebo-joint-position-controller-system" name="ignition::gazebo::systems::JointPositionController">
-            <joint_name>joint_art2_art3_pitch</joint_name>
-        </plugin>
-    </gazebo>
-    <gazebo>
-        <plugin filename="ignition-gazebo-joint-position-controller-system" name="ignition::gazebo::systems::JointPositionController">
-            <joint_name>joint_art3_art4_roll</joint_name>
-        </plugin>
-    </gazebo>
-    <gazebo>
-        <plugin filename="ignition-gazebo-joint-position-controller-system" name="ignition::gazebo::systems::JointPositionController">
-            <joint_name>joint_art4_art5_pitch</joint_name>
-        </plugin>
-    </gazebo>
-    <gazebo>
-        <plugin filename="ignition-gazebo-joint-position-controller-system" name="ignition::gazebo::systems::JointPositionController">
-            <joint_name>joint_art5_art6_roll</joint_name>
-        </plugin>
-    </gazebo>
-    <gazebo>
-        <plugin filename="ignition-gazebo-joint-position-controller-system" name="ignition::gazebo::systems::JointPositionController">
-            <joint_name>joint_arm_hand</joint_name>
-        </plugin>
-    </gazebo>
-    <gazebo>
-        <plugin filename="ignition-gazebo-joint-position-controller-system" name="ignition::gazebo::systems::JointPositionController">
-            <joint_name>joint_hand_finger_left</joint_name>
-        </plugin>
-    </gazebo>
-    <gazebo>
-        <plugin filename="ignition-gazebo-joint-position-controller-system" name="ignition::gazebo::systems::JointPositionController">
-            <joint_name>joint_hand_finger_right</joint_name>
-        </plugin>
-    </gazebo>
 </robot>
